File: OpenEarable-PCB-main-2.0/OpenEarable-PCB-main-2.0/OpenEarable-PCB-main-2.0.kicad_sch (KiCad schematic)
At the start: 0 parts

Commit message: modules in schem
Parts:
- added BT2: Battery_Cell, symbol Device:Battery_Cell
- added P1: USB_C_Plug_USB2.0, symbol Connector:USB_C_Plug_USB2.0
- added U1: MCP73831-2-OT, Package_TO_SOT_SMD:SOT-23-5, symbol Battery_Management:MCP73831-2-OT
- added U2: TPS22917DBV, Package_TO_SOT_SMD:SOT-23-6, symbol Power_Management:TPS22917DBV
- added U3, U4: TPS7A20xxxDQN, Package_SON:Texas_X2SON-4_1x1mm_P0.65mm, symbol Regulator_Linear:TPS7A20xxxDQN
- added U5: TPS3839DBZ, Package_TO_SOT_SMD:SOT-23, symbol Power_Supervisor:TPS3839DBZ
- added U6: BMI088, Package_LGA:Bosch_LGA-16_4.5x3mm_P0.5mm_LayoutBorder7x1y_ClockwisePinNumbering, symbol Sensor_Motion:BMI088
- added U7: NINA-B306-00B-00, XCVR_NINA-B306-00B-00, symbol NINA-B306-00B-00:NINA-B306-00B-00
- added U8: DRV2605LDGS, Package_SO:VSSOP-10_3x3mm_P0.5mm, symbol Driver_Haptic:DRV2605LDGS
Connections:
- new net: U7.12 (GND), U7.14 (GND), U7.26 (GND), U7.30 (GND), U7.53 (GND), U7.6 (GND)
- new net: U7.EAGP1 (EAGP), U7.EAGP2 (EAGP), U7.EAGP3 (EAGP), U7.EAGP4 (EAGP)
- new net: U7.EGP1 (EGP), U7.EGP10 (EGP), U7.EGP11 (EGP), U7.EGP12 (EGP), U7.EGP2 (EGP), U7.EGP3 (EGP), U7.EGP4 (EGP), U7.EGP5 (EGP), U7.EGP6 (EGP), U7.EGP7 (EGP), U7.EGP8 (EGP), U7.EGP9 (EGP)
- new net: P1.A1 (GND), P1.A12 (GND), P1.B1 (GND), P1.B12 (GND)
- new net: P1.A4 (VBUS), P1.A9 (VBUS), P1.B4 (VBUS), P1.B9 (VBUS)
- new net: U6.2 (GNDA), U6.4 (GNDA)
Other:
- title: (none) -> Main PCB
